File: CoulombCounter.sch (KiCad schematic (older format))
At the start: 10 parts, among them J1 Screw_Terminal_01x02, J2 Screw_Terminal_01x02, J3 Screw_Terminal_01x02

Commit message: Created PCB
Parts:
- 1u1: renamed from 1u; footprint (none) -> Capacitor_SMD:C_0805_2012Metric_Pad1.18x1.45mm_HandSolder
- 2k1, 2k2, 2k3: renamed from 2k; footprint (none) -> Resistor_SMD:R_0805_2012Metric_Pad1.20x1.40mm_HandSolder
- 50m1: renamed from 50m; footprint (none) -> Resistor_SMD:R_2512_6332Metric_Pad1.40x3.35mm_HandSolder
- J1, J2, J3: footprint (none) -> TerminalBlock_Phoenix:TerminalBlock_Phoenix_PT-1,5-2-3.5-H_1x02_P3.50mm_Horizontal
- J4: renamed from J?; footprint (none) -> Connector_PinHeader_2.54mm:PinHeader_1x05_P2.54mm_Vertical
- U1: renamed from U?; footprint (none) -> Package_DFN_QFN:DFN-8-1EP_3x3mm_P0.5mm_EP1.66x2.38mm
Connections:
- wire segments 28 -> 29
Other:
- moved on the sheet: 1u1, 2k1, 2k2, 2k3, 50m1, J1, J2, J3, J4, U1

Commit message: Fixed shorting PWR and GND, references and values, and silkscreen
Changed lines of the file:
@@
 $EndComp
 Connection ~ 5950 4300
-Wire Wire Line
-	4150 3500 4600 3500
 Text Label 4300 3900 0    50   ~ 0
 ~ALCC~
-Text Label 4150 3500 0    50   ~ 0
-+3.3V
+$Comp
+L power:+3.3V #PWR0109
+U 1 1 5FE6BDA3
+P 4350 3500
+F 0 "#PWR0109" H 4350 3350 50  0001 C CNN
+F 1 "+3.3V" H 4365 3673 50  0000 C CNN
+F 2 "" H 4350 3500 50  0001 C CNN
+F 3 "" H 4350 3500 50  0001 C CNN
+	1    4350 3500
+	1    0    0    -1
+$EndComp
+Wire Wire Line
+	4350 3500 4600 3500
 $EndSCHEMATC
